File: prerelease versions/Heawood-cornish/kicad/corne-heawood.kicad_sch (KiCad schematic)
At the start: 47 parts, among them J2 OLED, SW1 SW_PUSH, SW10 SW_PUSH, SW11 SW_PUSH, SW12 SW_PUSH, SW13 SW_PUSH, SW14 SW_PUSH, SW15 SW_PUSH, SW16 SW_PUSH, SW17 SW_PUSH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

Commit message: Add QMK firmware files
Parts:
- removed BATJ2: Conn_01x02_Female, Connector_JST:JST_PH_S2B-PH-K_1x02_P2.00mm_Horizontal, symbol Connector:Conn_01x02_Female
- added BatteryConnector1: ~, MyLibrary:2pad_battery_input, symbol my_symbol_library:battery_connector
- U2: footprint PCM_marbastlib-xp-promicroish:nice_nano_AH_USBup -> PCM_marbastlib-xp-promicroish:ProMicro_USBdn
Connections:
- net CS: now also U2.1 (P0.06); no longer U2.2 (P0.08)
- net GND: now also BatteryConnector1.1 (Batt-)
- net LED: now also U2.2 (P0.08); no longer U2.1 (P0.06)
- net at PSW1.3 (C): now also BatteryConnector1.2 (Batt+)
Changed lines of the file:
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@@
+    (stroke (width 0) (type default))
+  )
+  (wire (pts (xy 45.72 154.94) (xy 59.69 154.94))
     (stroke (width 0) (type default))
   )
@@
     (stroke (width 0) (type default))
   )
-  (wire (pts (xy 45.72 155.575) (xy 53.975 155.575))
-    (stroke (width 0) (type default))
-  )
-  (wire (pts (xy 45.72 140.97) (xy 45.72 155.575))
+  (wire (pts (xy 45.72 140.97) (xy 45.72 154.94))
     (stroke (width 0) (type default))
   )
@@
     (stroke (width 0) (type default))
   )
+  (wire (pts (xy 59.69 147.32) (xy 59.69 152.4))
+    (stroke (width 0) (type default))
+  )
   (wire (pts (xy 247.65 130.81) (xy 247.65 139.7))
     (stroke (width 0) (type default))
@@
     (stroke (width 0) (type default))
   )
+  (wire (pts (xy 83.82 76.2) (xy 88.9 76.2))
+    (stroke (width 0) (type default))
+  )
   (wire (pts (xy 240.03 157.48) (xy 222.25 157.48))
     (stroke (width 0) (type default))
@@
   )
   (wire (pts (xy 187.96 40.64) (xy 187.96 41.91))
+    (stroke (width 0) (type default))
+  )
+  (wire (pts (xy 83.82 78.74) (xy 88.9 78.74))
     (stroke (width 0) (type default))
   )
@@
     )
   )
-  (global_label "CS" (shape input) (at 88.9 78.74 180) (fields_autoplaced)
+  (global_label "CS" (shape input) (at 83.82 76.2 180) (fields_autoplaced)
     (effects (font (size 1.1938 1.1938)) (justify right))
-    (property "Intersheetrefs" "${INTERSHEET_REFS}" (at 84.3783 78.74 0)
+    (property "Intersheetrefs" "${INTERSHEET_REFS}" (at 79.2983 76.2 0)
       (effects (font (size 1.27 1.27)) (justify right) hide)
     )
@@
     )
   )
-  (global_label "LED" (shape input) (at 88.9 76.2 180) (fields_autoplaced)
+  (global_label "LED" (shape input) (at 83.82 78.74 180) (fields_autoplaced)
     (effects (font (size 1.1938 1.1938)) (justify right))
-    (property "Intersheetrefs" "${INTERSHEET_REFS}" (at 83.4688 76.2 0)
+    (property "Intersheetrefs" "${INTERSHEET_REFS}" (at 78.3888 78.74 0)
       (effects (font (size 1.27 1.27)) (justify right) hide)
     )
@@
     )
   )
-  (symbol (lib_id "Connector:Conn_01x02_Female") (at 59.055 155.575 0) (unit 1)
-    (in_bom yes) (on_board yes) (dnp no) (fields_autoplaced)
-    (property "Reference" "BATJ2" (at 59.7662 156.0103 0)
-      (effects (font (size 1.27 1.27)) (justify left))
-    )
-    (property "Value" "Conn_01x02_Female" (at 59.7662 158.5472 0)
-      (effects (font (size 1.27 1.27)) (justify left))
-    )
-    (property "Footprint" "Connector_JST:JST_PH_S2B-PH-K_1x02_P2.00mm_Horizontal" (at 59.055 155.575 0)
-      (effects (font (size 1.27 1.27)) hide)
-    )
-    (property "Datasheet" "~" (at 59.055 155.575 0)
-      (effects (font (size 1.27 1.27)) hide)
-    )
-    (pin "1")
-    (pin "2")
-    (instances
-      (project "corne-ultralight"
-        (path "/4d161fd0-88a3-46fc-b3eb-e2fe3659386b"
-          (reference "BATJ2") (unit 1)
-        )
-      )
-      (project "corne-heawood"
-        (path "/b2404ab0-025a-473e-9fbb-0abc932972cf"
-          (reference "BATJ2") (unit 1)
-        )
-      )
-    )
-  )
   (symbol (lib_id "PCM_marbastlib-promicroish:nice_nano") (at 107.95 90.17 0) (unit 1)
     (in_bom no) (on_board yes) (dnp no) (fields_autoplaced)
@@
       (effects (font (size 1.27 1.27)))
     )
-    (property "Footprint" "PCM_marbastlib-xp-promicroish:nice_nano_AH_USBup" (at 107.95 120.65 0)
+    (property "Footprint" "PCM_marbastlib-xp-promicroish:ProMicro_USBdn" (at 107.95 120.65 0)
       (effects (font (size 1.27 1.27)) hide)
     )
@@
     )
   )
+  (symbol (lib_id "my_symbol_library:battery_connector") (at 59.69 148.59 0) (unit 1)
+    (in_bom yes) (on_board yes) (dnp no) (fields_autoplaced)
+    (property "Reference" "BatteryConnector1" (at 69.85 153.67 0)
+      (effects (font (size 1.27 1.27)) (justify left))
+    )
+    (property "Value" "~" (at 59.69 148.59 0)
+      (effects (font (size 1.27 1.27)))
+    )
+    (property "Footprint" "MyLibrary:2pad_battery_input" (at 59.69 148.59 0)
+      (effects (font (size 1.27 1.27)) hide)
+    )
+    (property "Datasheet" "" (at 59.69 148.59 0)
+      (effects (font (size 1.27 1.27)) hide)
+    )
+    (pin "1")
+    (pin "2")
+    (instances
+      (project "corne-heawood"
+        (path "/b2404ab0-025a-473e-9fbb-0abc932972cf"
+          (reference "BatteryConnector1") (unit 1)
+        )
+      )
+    )
+  )
   (symbol (lib_id "PCM_marbastlib-various:SK6812MINI-E") (at 240.03 92.71 0) (unit 1)
     (in_bom yes) (on_board yes) (dnp no)
@@
     )
   )
-  (symbol (lib_id "power:GND") (at 53.975 158.115 0) (unit 1)
-    (in_bom yes) (on_board yes) (dnp no)
-    (property "Reference" "#PWR0109" (at 53.975 164.465 0)
-      (effects (font (size 1.27 1.27)) hide)
-    )
-    (property "Value" "GND" (at 53.975 161.925 0)
-      (effects (font (size 1.27 1.27)))
-    )
-    (property "Footprint" "" (at 53.975 158.115 0)
-      (effects (font (size 1.27 1.27)) hide)
-    )
-    (property "Datasheet" "" (at 53.975 158.115 0)
-      (effects (font (size 1.27 1.27)) hide)
-    )
+  (symbol (lib_id "power:GND") (at 59.69 147.32 180) (unit 1)
+    (in_bom yes) (on_board yes) (dnp no)
+    (property "Reference" "#PWR0109" (at 59.69 140.97 0)
+      (effects (font (size 1.27 1.27)) hide)
+    )
+    (property "Value" "GND" (at 59.69 143.51 0)
+      (effects (font (size 1.27 1.27)))
+    )
+    (property "Footprint" "" (at 59.69 147.32 0)
+      (effects (font (size 1.27 1.27)) hide)
+    )
+    (property "Datasheet" "" (at 59.69 147.32 0)
+      (effects (font (size 1.27 1.27)) hide)
+    )
